File: PCB/16x16/Bixel.sch (KiCad schematic (older format))
At the start: 263 parts, among them J1 Conn_01x12, J2 Conn_01x12, J3 Screw_Terminal_01x02, U1 74HC595, U2 74HC595

Commit message: Re-working schematic and layout for easier routing of LED power
Connections:
- net +5V: now also B112.5 (VCC), B128.8 (VCC), B144.5 (VCC), B16.5 (VCC), B160.8 (VCC), B176.5 (VCC), B192.8 (VCC), B208.5 (VCC), B224.8 (VCC), B240.5 (VCC), B256.8 (VCC), B32.8 (VCC), B48.5 (VCC), B64.8 (VCC), B80.5 (VCC), B96.8 (VCC)
- net GND: now also B113.1 (GND), B129.4 (GND), B145.1 (GND), B161.4 (GND), B17.1 (GND), B177.1 (GND), B193.4 (GND), B209.1 (GND), B225.4 (GND), B33.4 (GND), B49.1 (GND), B65.4 (GND), B81.1 (GND), B97.4 (GND)
Changed lines of the file:
@@
 $EndComp
 $Comp
-L bixel_up B128
-U 1 1 5B485074
-P 14600 20200
-F 0 "B128" V 14850 20000 60  0000 C CNN
-F 1 "bixel_up" V 14350 20050 39  0000 C CNN
-F 2 "custom:bixel" H 14600 20200 60  0001 C CNN
-F 3 "" H 14600 20200 60  0001 C CNN
-	1    14600 20200
-	1    0    0    -1
-$EndComp
-$Comp
 L bixel_down B129
 U 1 1 5B48F18A
@@
 Connection ~ 14200 3400
 Wire Wire Line
-	7800 20700 7800 21000
-Wire Wire Line
-	7800 21000 9050 21000
-Wire Wire Line
-	9050 21000 9050 20700
-Wire Wire Line
 	7900 20700 7900 20950
 Wire Wire Line
@@
 	8850 20900 8850 20700
 Wire Wire Line
-	8100 20700 8100 20850
-Wire Wire Line
-	8100 20850 8750 20850
-Wire Wire Line
-	8750 20850 8750 20700
-Wire Wire Line
-	9700 20700 9700 21000
-Wire Wire Line
-	9700 21000 10950 21000
-Wire Wire Line
-	10950 21000 10950 20700
-Wire Wire Line
 	9800 20700 9800 20950
 Wire Wire Line
@@
 	10750 20900 10750 20700
 Wire Wire Line
-	10000 20700 10000 20850
-Wire Wire Line
-	10000 20850 10650 20850
-Wire Wire Line
-	10650 20850 10650 20700
-Wire Wire Line
-	11600 20700 11600 21000
-Wire Wire Line
-	11600 21000 12850 21000
-Wire Wire Line
-	12850 21000 12850 20700
-Wire Wire Line
 	11700 20700 11700 20950
 Wire Wire Line
@@
 	12650 20900 12650 20700
 Wire Wire Line
-	11900 20700 11900 20850
-Wire Wire Line
-	11900 20850 12550 20850
-Wire Wire Line
-	12550 20850 12550 20700
-Wire Wire Line
-	13500 20700 13500 21000
-Wire Wire Line
-	13500 21000 14750 21000
-Wire Wire Line
-	14750 21000 14750 20700
-Wire Wire Line
 	13600 20700 13600 20950
 Wire Wire Line
@@
 	14550 20900 14550 20700
 Wire Wire Line
-	13800 20700 13800 20850
-Wire Wire Line
-	13800 20850 14450 20850
-Wire Wire Line
-	14450 20850 14450 20700
-Wire Wire Line
-	15400 20700 15400 21000
-Wire Wire Line
-	15400 21000 16650 21000
-Wire Wire Line
-	16650 21000 16650 20700
-Wire Wire Line
 	15500 20700 15500 20950
 Wire Wire Line
@@
 	16450 20900 16450 20700
 Wire Wire Line
-	15700 20700 15700 20850
-Wire Wire Line
-	15700 20850 16350 20850
-Wire Wire Line
-	16350 20850 16350 20700
-Wire Wire Line
-	17300 20700 17300 21000
-Wire Wire Line
-	17300 21000 18550 21000
-Wire Wire Line
-	18550 21000 18550 20700
-Wire Wire Line
 	17400 20700 17400 20950
 Wire Wire Line
@@
 	18350 20900 18350 20700
 Wire Wire Line
-	17600 20700 17600 20850
-Wire Wire Line
-	17600 20850 18250 20850
-Wire Wire Line
-	18250 20850 18250 20700
-Wire Wire Line
-	19200 20700 19200 21000
-Wire Wire Line
-	19200 21000 20450 21000
-Wire Wire Line
-	20450 21000 20450 20700
-Wire Wire Line
 	19300 20700 19300 20950
 Wire Wire Line
@@
 	20250 20900 20250 20700
 Wire Wire Line
-	19500 20700 19500 20850
-Wire Wire Line
-	19500 20850 20150 20850
-Wire Wire Line
-	20150 20850 20150 20700
-Wire Wire Line
-	21100 20700 21100 21000
-Wire Wire Line
-	21100 21000 22350 21000
-Wire Wire Line
-	22350 21000 22350 20700
-Wire Wire Line
 	21200 20700 21200 20950
 Wire Wire Line
@@
 	22150 20900 22150 20700
 Wire Wire Line
-	21400 20700 21400 20850
-Wire Wire Line
-	21400 20850 22050 20850
-Wire Wire Line
-	22050 20850 22050 20700
-Wire Wire Line
 	8750 2450 8750 2200
 Wire Wire Line
@@
 Text GLabel 25400 4600 0    51   Input ~ 0
 3V3
+Wire Wire Line
+	9050 20700 9050 21000
+Wire Wire Line
+	9050 21000 7800 21000
+Wire Wire Line
+	7800 21000 7800 20700
+Wire Wire Line
+	10950 20700 10950 21000
+Wire Wire Line
+	10950 21000 9700 21000
+Wire Wire Line
+	9700 21000 9700 20700
+Wire Wire Line
+	12850 20700 12850 21000
+Wire Wire Line
+	12850 21000 11600 21000
+Wire Wire Line
+	11600 21000 11600 20700
+$Comp
+L bixel_up B128
+U 1 1 5B485074
+P 14600 20200
+F 0 "B128" V 14850 20000 60  0000 C CNN
+F 1 "bixel_up" V 14350 20050 39  0000 C CNN
+F 2 "custom:bixel" H 14600 20200 60  0001 C CNN
+F 3 "" H 14600 20200 60  0001 C CNN
+	1    14600 20200
+	1    0    0    -1
+$EndComp
+Wire Wire Line
+	13500 20700 13500 21000
+Wire Wire Line
+	13500 21000 14750 21000
+Wire Wire Line
+	14750 21000 14750 20700
+Wire Wire Line
+	15400 20700 15400 21000
+Wire Wire Line
+	15400 21000 16650 21000
+Wire Wire Line
+	16650 21000 16650 20700
+Wire Wire Line
+	18550 20700 18550 21000
+Wire Wire Line
+	18550 21000 17300 21000
+Wire Wire Line
+	17300 21000 17300 20700
+Wire Wire Line
+	22350 20700 22350 21000
+Wire Wire Line
+	22350 21000 21100 21000
+Wire Wire Line
+	21100 21000 21100 20700
+Wire Wire Line
+	20450 20700 20450 21000
+Wire Wire Line
+	20450 21000 19200 21000
+Wire Wire Line
+	19200 21000 19200 20700
+Text GLabel 9050 21000 2    60   Input ~ 0
+5V
+Text GLabel 10950 21000 2    60   Input ~ 0
+5V
+Text GLabel 12850 21000 2    60   Input ~ 0
+5V
+Text GLabel 14750 21000 2    60   Input ~ 0
+5V
+Text GLabel 16650 21000 2    60   Input ~ 0
+5V
+Text GLabel 18550 21000 2    60   Input ~ 0
+5V
+Text GLabel 20450 21000 2    60   Input ~ 0
+5V
+Text GLabel 22350 21000 2    60   Input ~ 0
+5V
+Wire Wire Line
+	19500 20700 19500 20850
+Wire Wire Line
+	19500 20850 20150 20850
+Wire Wire Line
+	20150 20850 20150 20700
+Wire Wire Line
+	21400 20700 21400 20850
+Wire Wire Line
+	21400 20850 22050 20850
+Wire Wire Line
+	22050 20850 22050 20700
+Wire Wire Line
+	18250 20700 18250 20850
+Wire Wire Line
+	18250 20850 17600 20850
+Wire Wire Line
+	17600 20850 17600 20700
+Wire Wire Line
+	15700 20700 15700 20850
+Wire Wire Line
+	15700 20850 16350 20850
+Wire Wire Line
+	16350 20850 16350 20700
+Wire Wire Line
+	14450 20700 14450 20850
+Wire Wire Line
+	14450 20850 13800 20850
+Wire Wire Line
+	13800 20850 13800 20700
+Wire Wire Line
+	11900 20700 11900 20850
+Wire Wire Line
+	11900 20850 12550 20850
+Wire Wire Line
+	12550 20850 12550 20700
+Wire Wire Line
+	10000 20700 10000 20850
+Wire Wire Line
+	10000 20850 10650 20850
+Wire Wire Line
+	10650 20850 10650 20700
+Wire Wire Line
+	8750 20700 8750 20850
+Wire Wire Line
+	8750 20850 8100 20850
+Wire Wire Line
+	8100 20850 8100 20700
+Text GLabel 8750 2200 0    60   Input ~ 0
+GND
+Text GLabel 10650 2200 0    60   Input ~ 0
+GND
+Text GLabel 12550 2200 0    60   Input ~ 0
+GND
+Text GLabel 14450 2200 0    60   Input ~ 0
+GND
+Text GLabel 16350 2200 0    60   Input ~ 0
+GND
+Text GLabel 18250 2200 0    60   Input ~ 0
+GND
+Text GLabel 20150 2200 0    60   Input ~ 0
+GND
 $EndSCHEMATC
