File: PCB/ControlCarrier/ControlCarrier.sch (KiCad schematic (older format))
At the start: 7 parts, among them J1 RPi_GPIO, P2 CONN_01X02, U1 74AHC125

Commit message: Adding controller carrier
Parts:
- removed J?: Conn_02x12_Top_Bottom, symbol Conn_02x12_Top_Bottom
- added J2: Conn_02x12_Odd_Even, Socket_Strips:Socket_Strip_Straight_2x12_Pitch2.54mm, symbol Conn_02x12_Odd_Even
- added J3: Conn_02x03_Odd_Even, symbol Conn_02x03_Odd_Even
- C1, C2: renamed from C?; footprint (none) -> Capacitors_THT:CP_Radial_D10.0mm_P5.00mm
- U2: renamed from U?; footprint (none) -> teensy:Teensy35_36_NoCenterPins
Connections:
- net GND: now also P2.2 (Pin_2), J2.12 (Pin_12), J3.2 (Pin_2), J3.4 (Pin_4), J3.6 (Pin_6); no longer P2.1 (Pin_1)
- net LED_CLK: now also J2.16 (Pin_16)
- net LED_MOSI: now also J2.14 (Pin_14)
- net ROW_0: now also J2.18 (Pin_18)
- net ROW_1: now also J2.20 (Pin_20)
- net ROW_10: now also J2.11 (Pin_11)
- net ROW_11: now also J2.9 (Pin_9)
- net ROW_12: now also J2.7 (Pin_7)
- net ROW_13: now also J2.5 (Pin_5)
- net ROW_14: now also J2.3 (Pin_3)
- net ROW_15: now also J2.1 (Pin_1)
- net ROW_2: now also J2.22 (Pin_22)
- net ROW_3: now also J2.24 (Pin_24)
- net ROW_4: now also J2.23 (Pin_23)
- net ROW_5: now also J2.21 (Pin_21)
- net ROW_6: now also J2.19 (Pin_19)
- net ROW_7: now also J2.17 (Pin_17)
- net ROW_8: now also J2.15 (Pin_15)
- net ROW_9: now also J2.13 (Pin_13)
- net SHIFT_CLOCK: now also J2.8 (Pin_8)
- net SHIFT_DATA: now also J2.6 (Pin_6)
- net SHIFT_LATCH: now also J2.10 (Pin_10)
- net at J1.36 (GPIO16): now also J3.1 (Pin_1)
- net at J1.38 (GPIO20): now also J3.3 (Pin_3)
- net at J1.40 (GPIO21): now also J3.5 (Pin_5)
- net 5V renamed +5V
- net +5V: now also P2.1 (Pin_1); no longer P2.2 (Pin_2)
- net TEENSY_3V3 renamed +3V3
- net +3V3: now also J2.4 (Pin_4)
- no-connect marks 33 -> 97
Changed lines of the file:
@@
 Text GLabel 4000 2800 0    31   Input ~ 0
 GND
-Text GLabel 4350 1500 2    31   Input ~ 0
+Text GLabel 4350 1600 2    31   Input ~ 0
 5V
 Text GLabel 4000 3100 0    31   Input ~ 0
@@
 	-1   0    0    1
 $EndComp
-Text GLabel 4350 1600 2    31   Input ~ 0
+Text GLabel 4350 1500 2    31   Input ~ 0
 GND
 Text GLabel 1600 3950 0    31   Input ~ 0
@@
 NoConn ~ 1600 3750
 NoConn ~ 1600 3850
-NoConn ~ 3500 3950
-NoConn ~ 3500 3850
 NoConn ~ 3500 3550
-NoConn ~ 3500 3750
 NoConn ~ 3500 2850
 NoConn ~ 1600 2650
@@
 NoConn ~ 3500 2550
 NoConn ~ 1600 3650
-$Comp
-L Conn_02x12_Top_Bottom J?
-U 1 1 5B524153
-P 6750 2850
-F 0 "J?" H 6800 3450 50  0000 C CNN
-F 1 "Conn_02x12_Top_Bottom" H 6800 2150 50  0000 C CNN
-F 2 "" H 6750 2850 50  0001 C CNN
-F 3 "" H 6750 2850 50  0001 C CNN
-	1    6750 2850
-	1    0    0    -1
-$EndComp
-Text GLabel 6550 2350 0    31   Input ~ 0
+Text GLabel 6850 2350 2    31   Input ~ 0
 ROW_15
-Text GLabel 6550 2450 0    31   Input ~ 0
+Text GLabel 6850 2450 2    31   Input ~ 0
 ROW_14
-Text GLabel 6550 2550 0    31   Input ~ 0
+Text GLabel 6850 2550 2    31   Input ~ 0
 ROW_13
-Text GLabel 6550 2650 0    31   Input ~ 0
+Text GLabel 6850 2650 2    31   Input ~ 0
 ROW_12
-Text GLabel 6550 2750 0    31   Input ~ 0
+Text GLabel 6850 2750 2    31   Input ~ 0
 ROW_11
-Text GLabel 6550 2850 0    31   Input ~ 0
+Text GLabel 6850 2850 2    31   Input ~ 0
 ROW_10
-Text GLabel 6550 2950 0    31   Input ~ 0
+Text GLabel 6850 2950 2    31   Input ~ 0
 ROW_9
-Text GLabel 6550 3050 0    31   Input ~ 0
+Text GLabel 6850 3050 2    31   Input ~ 0
 ROW_8
-Text GLabel 6550 3150 0    31   Input ~ 0
+Text GLabel 6850 3150 2    31   Input ~ 0
 ROW_7
-Text GLabel 6550 3250 0    31   Input ~ 0
+Text GLabel 6850 3250 2    31   Input ~ 0
 ROW_6
-Text GLabel 6550 3350 0    31   Input ~ 0
+Text GLabel 6850 3350 2    31   Input ~ 0
 ROW_5
-Text GLabel 6550 3450 0    31   Input ~ 0
+Text GLabel 6850 3450 2    31   Input ~ 0
 ROW_4
-Text GLabel 7050 3450 2    31   Input ~ 0
+Text GLabel 6350 3450 0    31   Input ~ 0
 ROW_3
-Text GLabel 7050 3350 2    31   Input ~ 0
+Text GLabel 6350 3350 0    31   Input ~ 0
 ROW_2
-Text GLabel 7050 3250 2    31   Input ~ 0
+Text GLabel 6350 3250 0    31   Input ~ 0
 ROW_1
-Text GLabel 7050 3150 2    31   Input ~ 0
+Text GLabel 6350 3150 0    31   Input ~ 0
 ROW_0
-NoConn ~ 7050 2350
-Text GLabel 7050 3050 2    31   Input ~ 0
+NoConn ~ 6350 2350
+Text GLabel 6350 3050 0    31   Input ~ 0
 LED_CLK
-Text GLabel 7050 2950 2    31   Input ~ 0
+Text GLabel 6350 2950 0    31   Input ~ 0
 LED_MOSI
-Text GLabel 7050 2850 2    31   Input ~ 0
-GND
-Text GLabel 7050 2750 2    31   Input ~ 0
+Text GLabel 6350 2850 0    31   Input ~ 0
+GND
+Text GLabel 6350 2750 0    31   Input ~ 0
 SHIFT_LATCH
-Text GLabel 7050 2650 2    31   Input ~ 0
+Text GLabel 6350 2650 0    31   Input ~ 0
 SHIFT_CLOCK
-Text GLabel 7050 2550 2    31   Input ~ 0
+Text GLabel 6350 2550 0    31   Input ~ 0
 SHIFT_DATA
-Text GLabel 7050 2450 2    31   Input ~ 0
+Text GLabel 6350 2450 0    31   Input ~ 0
 TEENSY_3V3
 Text GLabel 5300 2850 2    31   Input ~ 0
@@
 LED_MOSI
 $Comp
-L Teensy3.6 U?
+L Teensy3.6 U2
 U 1 1 5B524C9F
 P 9150 3250
-F 0 "U?" H 9150 5550 60  0000 C CNN
+F 0 "U2" H 9150 5550 60  0000 C CNN
 F 1 "Teensy3.6" H 9150 950 60  0000 C CNN
-F 2 "" H 9150 3250 60  0000 C CNN
+F 2 "teensy:Teensy35_36_NoCenterPins" H 9150 3250 60  0001 C CNN
 F 3 "" H 9150 3250 60  0000 C CNN
 	1    9150 3250
@@
 GND
 $Comp
-L CP C?
+L CP C1
 U 1 1 5B525C03
 P 4950 1550
-F 0 "C?" H 4975 1650 50  0000 L CNN
+F 0 "C1" H 4975 1650 50  0000 L CNN
 F 1 "1000uF" H 4975 1450 50  0000 L CNN
-F 2 "" H 4988 1400 50  0001 C CNN
+F 2 "Capacitors_THT:CP_Radial_D10.0mm_P5.00mm" H 4988 1400 50  0001 C CNN
 F 3 "" H 4950 1550 50  0001 C CNN
 	1    4950 1550
@@
 $EndComp
 $Comp
-L CP C?
+L CP C2
 U 1 1 5B525C51
 P 5300 1550
-F 0 "C?" H 5325 1650 50  0000 L CNN
+F 0 "C2" H 5325 1650 50  0000 L CNN
 F 1 "1000uF" H 5325 1450 50  0000 L CNN
-F 2 "" H 5338 1400 50  0001 C CNN
+F 2 "Capacitors_THT:CP_Radial_D10.0mm_P5.00mm" H 5338 1400 50  0001 C CNN
 F 3 "" H 5300 1550 50  0001 C CNN
 	1    5300 1550
@@
 $EndComp
 Wire Wire Line
-	4950 1700 5300 1700
-Wire Wire Line
-	4950 1400 5300 1400
+	4750 1700 5300 1700
+Wire Wire Line
+	4750 1400 5300 1400
 Text GLabel 4950 1400 1    31   Input ~ 0
 5V
 Text GLabel 4950 1700 3    31   Input ~ 0
 GND
+NoConn ~ 8150 3350
+NoConn ~ 8150 3450
+NoConn ~ 8150 3550
+NoConn ~ 8150 3650
+NoConn ~ 8150 3750
+NoConn ~ 8150 3850
+NoConn ~ 8150 3950
+NoConn ~ 8150 4050
+NoConn ~ 8150 4150
+NoConn ~ 8150 4250
+NoConn ~ 8150 4350
+NoConn ~ 8150 4450
+NoConn ~ 8150 4550
+NoConn ~ 8150 4650
+NoConn ~ 8150 4750
+NoConn ~ 8150 4850
+NoConn ~ 8150 5050
+NoConn ~ 8150 5150
+NoConn ~ 8150 5250
+NoConn ~ 8150 5350
+NoConn ~ 10150 5350
+NoConn ~ 10150 5250
+NoConn ~ 10150 5150
+NoConn ~ 10150 5050
+NoConn ~ 10150 4950
+NoConn ~ 10150 4850
+NoConn ~ 10150 4750
+NoConn ~ 10150 4550
+NoConn ~ 10150 4450
+NoConn ~ 10150 4350
+NoConn ~ 10150 4250
+NoConn ~ 10150 4150
+NoConn ~ 10150 4050
+NoConn ~ 10150 3950
+NoConn ~ 10150 3850
+NoConn ~ 10150 3750
+NoConn ~ 10150 3650
+NoConn ~ 10150 3550
+NoConn ~ 10150 3450
+NoConn ~ 10150 3350
+NoConn ~ 10150 3250
+NoConn ~ 10150 3150
+NoConn ~ 10150 3050
+NoConn ~ 10150 2950
+NoConn ~ 10150 2850
+NoConn ~ 10150 2750
+NoConn ~ 10150 2650
+NoConn ~ 10150 2550
+NoConn ~ 10150 2450
+NoConn ~ 10150 2350
+NoConn ~ 10150 2250
+NoConn ~ 10150 2150
+NoConn ~ 10150 2050
+NoConn ~ 10150 1950
+NoConn ~ 10150 1850
+NoConn ~ 10150 1750
+NoConn ~ 10150 1650
+NoConn ~ 10150 1550
+NoConn ~ 10150 1450
+NoConn ~ 10150 1350
+NoConn ~ 10150 1250
+NoConn ~ 10150 1150
+NoConn ~ 10350 2550
+NoConn ~ 10350 2400
+NoConn ~ 8150 1550
+NoConn ~ 8150 2550
+NoConn ~ 3650 3250
+$Comp
+L +3.3V #PWR01
+U 1 1 5B526F2E
+P 10300 4550
+F 0 "#PWR01" H 10300 4400 50  0001 C CNN
+F 1 "+3.3V" H 10300 4690 50  0000 C CNN
+F 2 "" H 10300 4550 50  0001 C CNN
+F 3 "" H 10300 4550 50  0001 C CNN
+	1    10300 4550
+	1    0    0    -1
+$EndComp
+Wire Wire Line
+	10300 4550 10300 4600
+Wire Wire Line
+	10300 4600 10150 4600
+Wire Wire Line
+	10150 4600 10150 4650
+$Comp
+L +5V #PWR02
+U 1 1 5B52707B
+P 4750 1400
+F 0 "#PWR02" H 4750 1250 50  0001 C CNN
+F 1 "+5V" H 4750 1540 50  0000 C CNN
+F 2 "" H 4750 1400 50  0001 C CNN
+F 3 "" H 4750 1400 50  0001 C CNN
+	1    4750 1400
+	0    -1   -1   0
+$EndComp
+$Comp
+L GND #PWR03
+U 1 1 5B52709D
+P 4750 1700
+F 0 "#PWR03" H 4750 1450 50  0001 C CNN
+F 1 "GND" H 4750 1550 50  0000 C CNN
+F 2 "" H 4750 1700 50  0001 C CNN
+F 3 "" H 4750 1700 50  0001 C CNN
+	1    4750 1700
+	0    1    1    0
+$EndComp
+Connection ~ 4950 1700
+Connection ~ 4950 1400
+$Comp
+L Conn_02x12_Odd_Even J2
+U 1 1 5B525CAD
+P 6650 2850
+F 0 "J2" H 6700 3450 50  0000 C CNN
+F 1 "Conn_02x12_Odd_Even" H 6700 2150 50  0000 C CNN
+F 2 "Socket_Strips:Socket_Strip_Straight_2x12_Pitch2.54mm" H 6650 2850 50  0001 C CNN
+F 3 "" H 6650 2850 50  0001 C CNN
+	1    6650 2850
+	-1   0    0    -1
+$EndComp
+Wire Wire Line
+	3500 3750 3700 3750
+Wire Wire Line
+	3700 3850 3500 3850
+Wire Wire Line
+	3500 3950 3700 3950
+Wire Wire Line
+	4200 3750 4200 3950
+Connection ~ 4200 3850
+Text GLabel 4200 3850 2    31   Input ~ 0
+GND
+$Comp
+L Conn_02x03_Odd_Even J3
+U 1 1 5B527992
+P 3900 3850
+F 0 "J3" H 3950 4050 50  0000 C CNN
+F 1 "Conn_02x03_Odd_Even" H 3950 3650 50  0000 C CNN
+F 2 "" H 3900 3850 50  0001 C CNN
+F 3 "" H 3900 3850 50  0001 C CNN
+	1    3900 3850
+	1    0    0    -1
+$EndComp
 $EndSCHEMATC
